File: STPMIC1_MC32PF3000_Board/STPMIC1_MC32PF3000_Board/PF3000.sch (KiCad schematic (older format))
At the start: 65 parts, among them U2 PF3000

Commit message: Completed RevA layout
Parts:
- C26, C27, C28, C29, C30, C33, C37, C38, C41, C42, C43, C50, C53, C54, C55: footprint Capacitor_SMD:C_0402_1005Metric_Pad0.74x0.62mm_HandSolder -> Capacitor_SMD:C_0805_2012Metric_Pad1.18x1.45mm_HandSolder
- C31, C32, C34, C35, C36, C39, C40: footprint Capacitor_SMD:C_0402_1005Metric_Pad0.74x0.62mm_HandSolder -> Capacitor_SMD:C_0805_2012Metric_Pad1.18x1.45mm_HandSolder; Type CAP CER 1.0UF 10V 10% X5R 0402 -> (none)
- C44, C46: MfrNum (none) -> CL21A226MPQNNNE; Type CAP CER 2.2UF 6.3V 20% X5R 0402 -> CAP CER 22uF 25V 20% X5R 0805
- C49: footprint Capacitor_SMD:C_0402_1005Metric_Pad0.74x0.62mm_HandSolder -> Capacitor_SMD:C_0805_2012Metric_Pad1.18x1.45mm_HandSolder; MfrNum (none) -> CL21A226MPQNNNE; Type CAP CER 2.2UF 6.3V 20% X5R 0402 -> CAP CER 22uF 25V 20% X5R 0805
- C51: footprint Capacitor_SMD:C_0402_1005Metric_Pad0.74x0.62mm_HandSolder -> Capacitor_SMD:C_0805_2012Metric_Pad1.18x1.45mm_HandSolder; Type CAP CER 470nF 10V 10% X7R 0402 -> (none)
- C52: footprint Capacitor_SMD:C_0402_1005Metric_Pad0.74x0.62mm_HandSolder -> Capacitor_SMD:C_0603_1608Metric_Pad1.08x0.95mm_HandSolder
- C56, C57, C58, C59, C60, C61, C62, C63, C64, C65: MfrNum (none) -> CL21A226MPQNNNE
- C66: footprint Capacitor_SMD:C_0402_1005Metric_Pad0.74x0.62mm_HandSolder -> Capacitor_SMD:C_0805_2012Metric_Pad1.18x1.45mm_HandSolder; Type CAP CER 10nF 50V 10% X7R 0402 -> (none)
- NT1, NT10, NT11, NT12, NT13, NT14, NT2, NT3, NT4, NT5, NT6, NT7, NT8, NT9: footprint NetTie:NetTie-2_SMD_Pad0.5mm -> TinyNetTies:NetTie-2_SMD_Pad0.254mm

Commit message: Completed RevA
Parts:
- C26, C27, C28, C33, C41, C48, C53, C55: LCSC (none) -> C28323
- C29, C30, C37, C38, C42, C67: LCSC (none) -> C15850
- C31, C32, C34, C35, C36, C39, C40: LCSC (none) -> C49678
- C43, C45, C47, C50: LCSC (none) -> C1779
- C44, C46, C49, C56, C57, C58, C59, C60, C61, C62, C63, C64, C65: LCSC (none) -> C45783
- C51: LCSC (none) -> C13967
- C52: footprint Capacitor_SMD:C_0603_1608Metric_Pad1.08x0.95mm_HandSolder -> Capacitor_SMD:C_0805_2012Metric_Pad1.18x1.45mm_HandSolder; LCSC (none) -> C5378
- C54: LCSC (none) -> C5378
- C66: LCSC (none) -> C1710
- D16: LCSC (none) -> C190475
- L10: footprint Inductor_SMD:L_1008_2520Metric_Pad1.43x2.20mm_HandSolder -> Inductor_SMD:L_Coilcraft_LPS4018; Mouser (none) -> 994-LPS4018-222MRC
- L6, L7, L8, L9: Mouser (none) -> 81-DFE252012P-1R5MP2; Type IND PWR 1.5uH@1MHz 3.5A 20% 2520 -> IND PWR 1.5uH@1MHz 3.5A 20% 1008
- R20, R21: LCSC (none) -> C17414
- U2: MfrNum (none) -> MC32PF3000A8EP; Mouser (none) -> 841-MC32PF3000A8EP
