File: STPMIC1_MC32PF3000_Board/STPMIC1_MC32PF3000_Board/PF3000_Board.sch (KiCad schematic (older format))
At the start: 33 parts, among them J12 Conn_01x02, J13 Conn_01x03, J14 Conn_01x03, J15 Barrel_Jack_Switch, J16 Conn_01x03, J17 Conn_01x03, J18 Conn_01x03, J19 Conn_01x02, J20 Conn_01x03, J21 Conn_02x13_Odd_Even, J22 Conn_01x03, Q1 FDMA908PZ, Q2 Q_PMOS_DGS, Q3 Q_PMOS_DGS, SW5 SW_SPST, U3 SE8233X2

Commit message: Completed RevA layout
Parts:
- removed Q2, Q3: Q_PMOS_DGS, symbol Device:Q_PMOS_DGS
- added D19, D20, D21, D22, D23, D24, D25, D26, D27, D28, D29, D30, D31: D, Diode_SMD:D_0805_2012Metric_Pad1.15x1.40mm_HandSolder, symbol Device:D
- added Q2, Q3: Q_PMOS_GSD, Package_TO_SOT_SMD:SOT-23, symbol Device:Q_PMOS_GSD
- added R29, R30, R31, R32, R33, R34, R35, R36, R37, R38, R39, R40, R41: 2K2, Resistor_SMD:R_0805_2012Metric_Pad1.20x1.40mm_HandSolder, symbol Device:R
- added TP15, TP16, TP17, TP18, TP19, TP20, TP21, TP22, TP23, TP24, TP25, TP26, TP27: TestPoint, TestPoint:TestPoint_Pad_D1.0mm, symbol Connector:TestPoint
- BT1: footprint (none) -> Battery:BatteryHolder_Seiko_MS621F
- C70, C71: footprint (none) -> Capacitor_SMD:C_0805_2012Metric_Pad1.18x1.45mm_HandSolder; MfrNum (none) -> C2012X5R1A476M125AC; Type (none) -> CAP CER 47uF 10V 20% X5R 0805
- C72, C73: footprint (none) -> Capacitor_SMD:C_0805_2012Metric_Pad1.18x1.45mm_HandSolder; MfrNum (none) -> CL21A226MPQNNNE; Type (none) -> CAP CER 22uF 25V 20% X5R 0805
- D17: footprint (none) -> LED_SMD:LED_0805_2012Metric_Pad1.15x1.40mm_HandSolder
- D18: footprint (none) -> LED_SMD:LED_0805_2012Metric_Castellated
- J15: footprint (none) -> Connector_BarrelJack:BarrelJack_Horizontal
- J21: footprint (none) -> Connector_PinHeader_2.54mm:PinHeader_2x13_P2.54mm_Vertical
- SW5: footprint (none) -> Button_Switch_SMD:SW_Push_1P1T_NO_CK_KMR2
- gave numbers to parts that had none: 1
Connections:
- net GNDS: now also D19.1 (K), D20.1 (K), D21.1 (K), D22.1 (K), D23.1 (K), D24.1 (K), D25.1 (K), D26.1 (K), D27.1 (K), D28.1 (K), D29.1 (K), D30.1 (K), D31.1 (K)
- net INTB: now also J23.5 (Pin_5), Q3.1 (G); no longer J23.6 (Pin_6)
- net LDO1_OUT: now also J21.25 (Pin_25), R33.1, TP19.1; no longer J21.9 (Pin_9)
- net LDO2_OUT: now also J21.23 (Pin_23), R34.1, TP20.1; no longer J21.11 (Pin_11)
- net LDO3_OUT: now also J21.19 (Pin_19), R35.1, TP21.1; no longer J21.13 (Pin_13)
- net LDO4_OUT: now also J21.17 (Pin_17), R36.1, TP22.1; no longer J21.15 (Pin_15)
- net PWRON: now also J23.6 (Pin_6); no longer J23.4 (Pin_4)
- net RESETBMCU: now also J23.3 (Pin_3), Q2.1 (G); no longer J23.5 (Pin_5)
- net SD_VSEL: now also J23.4 (Pin_4); no longer J23.3 (Pin_3)
- net SW1A_OUT: now also J21.3 (Pin_3), R29.1, TP15.1; no longer J21.1 (Pin_1)
- net SW1B_OUT: now also J21.1 (Pin_1), R30.1, TP16.1; no longer J21.3 (Pin_3)
- net SW2_OUT: now also J21.21 (Pin_21), R31.1, TP17.1; no longer J21.5 (Pin_5)
- net SW3_OUT: now also J21.13 (Pin_13), R32.1, TP18.1; no longer J21.7 (Pin_7)
- net SWBST_OUT: now also J21.5 (Pin_5), R37.1, TP23.1; no longer J21.17 (Pin_17)
- net V33_OUT: now also J21.11 (Pin_11), R41.1, TP27.1; no longer J21.25 (Pin_25)
- net VCCSD_OUT: now also J21.9 (Pin_9), R39.1, TP25.1; no longer J21.21 (Pin_21)
- net VREFDDR_OUT: now also J21.15 (Pin_15), R38.1, TP24.1; no longer J21.19 (Pin_19)
- net VSNVS_OUT: now also J21.7 (Pin_7), R40.1, TP26.1; no longer J21.23 (Pin_23)
- net V_PU: now also Q2.2 (S), Q3.2 (S)
- net at D17.2 (A): now also Q2.3 (D)
- net at D18.2 (A): now also Q3.3 (D)
- new net: D22.2 (A), R32.2
- new net: D19.2 (A), R29.2
- new net: D20.2 (A), R30.2
- new net: D21.2 (A), R31.2
- new net: D23.2 (A), R33.2
- new net: D24.2 (A), R34.2
- new net: D25.2 (A), R35.2
- new net: D26.2 (A), R36.2
- new net: D27.2 (A), R37.2
- new net: D28.2 (A), R38.2
- new net: D31.2 (A), R41.2
- new net: D30.2 (A), R40.2
- new net: D29.2 (A), R39.2
Other:
- moved on the sheet: J13, J14, J16, J20, J21, J23

Commit message: updated RevA Layout
Connections:
- net VPWR: no longer J15.3
- no-connect marks 0 -> 1
Changed lines of the file:
@@
 	-1   0    0    1
 $EndComp
-Wire Wire Line
-	2400 2025 2700 2025
-Connection ~ 2400 2025
-Wire Wire Line
-	2400 2125 2400 2025
-Wire Wire Line
-	2150 2125 2400 2125
 $Comp
 L power:GNDS #PWR028
@@
 Text Label 2700 2025 2    50   ~ 0
 VPWR
-Wire Wire Line
-	2150 2025 2400 2025
 Text Notes 1300 1575 0    50   ~ 0
 3.7 V to 5.5 V Supply input (Default). \n\nShorts VPWR to ground when not used (pin 3-2)\n
@@
 Wire Wire Line
 	8375 2725 6025 2725
+Wire Wire Line
+	2150 2025 2700 2025
+NoConn ~ 2150 2125
 $EndSCHEMATC

Commit message: Completed RevA
Parts:
- added JP1, JP2: Jumper_NO_Small, Jumper:SolderJumper-2_P1.3mm_Open_RoundedPad1.0x1.5mm, symbol Device:Jumper_NO_Small
- BT1: footprint Battery:BatteryHolder_Seiko_MS621F -> Panasonic_ML_series:ML1220_F1BN; MfrNum (none) -> ML-1220/F1BN; Type (none) -> Panasonic 3V Lithium Manganese Dioxide Button Rechargeable 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
- C68: LCSC (none) -> C28323
- C69: LCSC (none) -> C15850
- C70, C71: LCSC (none) -> C16780
- C72, C73: LCSC (none) -> C45783
- D17, D18: LCSC (none) -> C84256
- D19, D20, D21, D22, D23, D24, D25, D26, D27, D28, D29, D30, D31: footprint Diode_SMD:D_0805_2012Metric_Pad1.15x1.40mm_HandSolder -> LED_SMD:LED_0805_2012Metric_Pad1.15x1.40mm_HandSolder; LCSC (none) -> C84256
- J12, J19: LCSC (none) -> ~ ~ ~ ~ ~ ~ ~ ~ ~ ~
- Q1: Mouser (none) -> 512-FDMA908PZ; Type (none) -> PMOS PowerTrench -12V, -12A, 12.5mΩ MicroFET-6
- Q2, Q3: MfrNum (none) -> NTR1P02LT3G; Mouser (none) -> 863-NTR1P02LT1G
- R22, R23, R24, R25, R26: LCSC (none) -> C17407
- R27, R28, R29, R30, R31, R32, R33, R34, R35, R36, R37, R38, R39, R40, R41: LCSC (none) -> C17520
- SW5: MfrNum (none) -> KMR221NGLFS; Mouser (none) -> 611-KMR221NGLFS; Type (none) -> Tactile Microminiature SMT Top Actuated
- U3: LCSC (none) -> C437587; MfrNum (none) -> SE8233X2
Connections:
- net INTB: now also JP2.1
- net RESETBMCU: now also JP1.1
- net VDBG: now also Q2.2 (S), Q3.2 (S), JP1.2, JP2.2
- net V_PU: no longer Q2.2 (S), Q3.2 (S)
Other:
- moved on the sheet: D18, Q3, R28
