File: STPMIC1_MC32PF3000_Board/STPMIC1_MC32PF3000_Board/STPMIC1_Board.sch (KiCad schematic (older format))
At the start: 45 parts, among them J1 Conn_01x02, J10 Conn_01x03, J11 Conn_02x14_Odd_Even, J2 Conn_01x02, J3 Conn_01x02, J4 USB_B_Micro, J5 Conn_01x06, J6 Conn_01x03, J7 Conn_01x03, J8 Conn_02x03_Odd_Even, J9 Conn_01x03, SW1 SW_SPST, SW2 SW_SPST, SW3 SW_SPST

Commit message: updated schema document
Connections:
- net sheet60878B3D/SCL renamed SCL
- net sheet60878B3D/SDA renamed SDA
Other:
- note added: "DEBUG OUTPUT"
- note added: "DIAGNOSTICS OUTPUT"
- note added: "OUTPUT POWER INDICATORS"
- note added: "POWER INPUT"
- note added: "POWER MANAGEMENT IC"
- note added: "POWER OUTPUT"
- note added: "SUBSYSTEM JUMPERS"
- moved on the sheet: D1, D10, D11, D12, D13, D14, D15, D2, D3, D4, D5, D6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

Commit message: Completed RevA layout
Parts:
- D1, D2: footprint Diode_SMD:D_0805_2012Metric_Pad1.15x1.40mm_HandSolder -> LED_SMD:LED_0805_2012Metric_Pad1.15x1.40mm_HandSolder
Changed lines of the file:
@@
 F 0 "D1" V 2646 4145 50  0000 R CNN
 F 1 "D" V 2555 4145 50  0000 R CNN
-F 2 "Diode_SMD:D_0805_2012Metric_Pad1.15x1.40mm_HandSolder" H 2600 4225 50  0001 C CNN
+F 2 "LED_SMD:LED_0805_2012Metric_Pad1.15x1.40mm_HandSolder" H 2600 4225 50  0001 C CNN
 F 3 "~" H 2600 4225 50  0001 C CNN
 	1    2600 4225
@@
 F 0 "D2" V 5271 10045 50  0000 R CNN
 F 1 "D" V 5180 10045 50  0000 R CNN
-F 2 "Diode_SMD:D_0805_2012Metric_Pad1.15x1.40mm_HandSolder" H 5225 10125 50  0001 C CNN
+F 2 "LED_SMD:LED_0805_2012Metric_Pad1.15x1.40mm_HandSolder" H 5225 10125 50  0001 C CNN
 F 3 "~" H 5225 10125 50  0001 C CNN
 	1    5225 10125

Commit message: updated RevA Layout
Parts:
- removed J4: USB_B_Micro, Connector_USB:USB_Micro-B_Molex-105017-0001, symbol Connector:USB_B_Micro
- added J4: Barrel_Jack, Connector_BarrelJack:BarrelJack_Horizontal, symbol Connector:Barrel_Jack
Connections:
- net GNDS: now also J4.2
- net VBAT: now also J4.1
- no-connect marks 4 -> 0
Changed lines of the file:
@@
 $EndComp
 Wire Wire Line
-	2625 2150 3075 2150
-Text Label 3075 2150 2    50   ~ 0
+	2375 2200 2825 2200
+Text Label 2825 2200 2    50   ~ 0
 VBAT
-NoConn ~ 2625 2350
-NoConn ~ 2625 2450
-NoConn ~ 2625 2550
-Wire Wire Line
-	2325 2750 2325 2850
+Wire Wire Line
+	2575 2400 2575 2500
 $Comp
 L power:GNDS #PWR?
 U 1 1 60878CA7
-P 2325 2850
+P 2575 2500
 AR Path="/60878CA7" Ref="#PWR?"  Part="1"
 AR Path="/6085A652/60878CA7" Ref="#PWR0109"  Part="1"
-F 0 "#PWR0109" H 2325 2600 50  0001 C CNN
-F 1 "GNDS" H 2330 2677 50  0000 C CNN
-F 2 "" H 2325 2850 50  0001 C CNN
-F 3 "" H 2325 2850 50  0001 C CNN
-	1    2325 2850
-	1    0    0    -1
-$EndComp
-NoConn ~ 2225 2750
-$Comp
-L Connector:USB_B_Micro J?
-U 1 1 60878C9B
-P 2325 2350
-AR Path="/60878C9B" Ref="J?"  Part="1"
-AR Path="/6085A652/60878C9B" Ref="J4"  Part="1"
-F 0 "J4" H 2382 2817 50  0000 C CNN
-F 1 "USB_B_Micro" H 2382 2726 50  0000 C CNN
-F 2 "Connector_USB:USB_Micro-B_Molex-105017-0001" H 2475 2300 50  0001 C CNN
-F 3 "https://www.molex.com/molex/products/part-detail/io_connectors/1050170001" H 2475 2300 50  0001 C CNN
-	1    2325 2350
+F 0 "#PWR0109" H 2575 2250 50  0001 C CNN
+F 1 "GNDS" H 2580 2327 50  0000 C CNN
+F 2 "" H 2575 2500 50  0001 C CNN
+F 3 "" H 2575 2500 50  0001 C CNN
+	1    2575 2500
 	1    0    0    -1
 $EndComp
@@
 Text Notes 7025 8800 0    118  ~ 0
 OUTPUT POWER INDICATORS
+$Comp
+L Connector:Barrel_Jack J4
+U 1 1 608BA36B
+P 2075 2300
+F 0 "J4" H 2132 2625 50  0000 C CNN
+F 1 "Barrel_Jack" H 2132 2534 50  0000 C CNN
+F 2 "Connector_BarrelJack:BarrelJack_Horizontal" H 2125 2260 50  0001 C CNN
+F 3 "~" H 2125 2260 50  0001 C CNN
+	1    2075 2300
+	1    0    0    -1
+$EndComp
+Wire Wire Line
+	2575 2400 2375 2400
+$Comp
+L power:PWR_FLAG #FLG0114
+U 1 1 608FAE9D
+P 2950 2500
+F 0 "#FLG0114" H 2950 2575 50  0001 C CNN
+F 1 "PWR_FLAG" H 2950 2673 50  0000 C CNN
+F 2 "" H 2950 2500 50  0001 C CNN
+F 3 "~" H 2950 2500 50  0001 C CNN
+	1    2950 2500
+	-1   0    0    1
+$EndComp
+Wire Wire Line
+	2950 2500 2950 2400
+Wire Wire Line
+	2950 2400 2575 2400
+Connection ~ 2575 2400
 $EndSCHEMATC

Commit message: Completed RevA
Parts:
- D1, D2: LCSC (none) -> C84256
- D10, D11, D12, D13, D14, D15, D3, D4, D5, D6, D7, D8, D9: footprint Diode_SMD:D_0805_2012Metric_Pad1.15x1.40mm_HandSolder -> LED_SMD:LED_0805_2012Metric_Pad1.15x1.40mm_HandSolder; LCSC (none) -> C84256
- J1, J2, J3: LCSC (none) -> ~ ~ ~ ~ ~ ~ ~ ~ ~ ~
- R1, R10, R11, R12, R13, R14, R15, R16, R2, R3, R4, R5, R6, R7, R8, R9: LCSC (none) -> C17520
- SW1, SW2, SW3: MfrNum (none) -> KMR221NGLFS; Mouser (none) -> 611-KMR221NGLFS; Type (none) -> Tactile Microminiature SMT Top Actuated
