File: STPMIC1_MC32PF3000_Board/STPMIC1_MC32PF3000_Board/STPMIC1_MC32PF3000_Board.kicad_pcb (KiCad board)
At the start: 4 copper layers, 99.1 x 99.1 mm, 93 parts, among them J1 Conn_01x02, J10 Conn_01x03, J11 Conn_02x14_Odd_Even, J2 Conn_01x02, J3 Conn_01x02, J4 USB_B_Micro, J5 Conn_01x06, J6 Conn_01x03, J7 Conn_01x03, J8 Conn_02x03_Odd_Even, J9 Conn_01x03, SW1 SW_SPST, SW2 SW_SPST, SW3 SW_SPST, U1 STPMIC1

Commit message: Completed RevA layout
Parts:
- added BT1: Battery_Cell, Battery:BatteryHolder_Seiko_MS621F, F.Cu at (132.1, 98.8)
- added C26: 1uF, Capacitor_SMD:C_0805_2012Metric_Pad1.18x1.45mm_HandSolder, F.Cu at (110.7, 124.0)
- added C27: 1uF, Capacitor_SMD:C_0805_2012Metric_Pad1.18x1.45mm_HandSolder, F.Cu at (114.7, 128.0)
- added C28: 1uF, Capacitor_SMD:C_0805_2012Metric_Pad1.18x1.45mm_HandSolder, F.Cu at (126.1, 124.3)
- added C29: 10uF, Capacitor_SMD:C_0805_2012Metric_Pad1.18x1.45mm_HandSolder, F.Cu at (116.1, 114.4)
- added C30: 10uF, Capacitor_SMD:C_0805_2012Metric_Pad1.18x1.45mm_HandSolder, F.Cu at (121.0, 124.5)
- added C31: 100nF, Capacitor_SMD:C_0805_2012Metric_Pad1.18x1.45mm_HandSolder, F.Cu at (114.0, 114.4)
- added C32: 100nF, Capacitor_SMD:C_0805_2012Metric_Pad1.18x1.45mm_HandSolder, F.Cu at (121.0, 122.4)
- added C33: 1uF, Capacitor_SMD:C_0805_2012Metric_Pad1.18x1.45mm_HandSolder, F.Cu at (141.4, 120.6)
- added C34: 100nF, Capacitor_SMD:C_0805_2012Metric_Pad1.18x1.45mm_HandSolder, F.Cu at (117.6, 109.6)
- added C35: 100nF, Capacitor_SMD:C_0805_2012Metric_Pad1.18x1.45mm_HandSolder, F.Cu at (132.2, 124.3)
- added C36: 100nF, Capacitor_SMD:C_0805_2012Metric_Pad1.18x1.45mm_HandSolder, F.Cu at (130.2, 124.3)
- added C37: 10uF, Capacitor_SMD:C_0805_2012Metric_Pad1.18x1.45mm_HandSolder, F.Cu at (116.1, 118.7)
- added C38: 10uF, Capacitor_SMD:C_0805_2012Metric_Pad1.18x1.45mm_HandSolder, F.Cu at (129.6, 118.3)
- added C39: 100nF, Capacitor_SMD:C_0805_2012Metric_Pad1.18x1.45mm_HandSolder, F.Cu at (114.0, 118.7)
- added C40: 100nF, Capacitor_SMD:C_0805_2012Metric_Pad1.18x1.45mm_HandSolder, F.Cu at (131.7, 118.3)
- added C41: 1uF, Capacitor_SMD:C_0805_2012Metric_Pad1.18x1.45mm_HandSolder, F.Cu at (123.7, 105.8)
- added C42: 10uF, Capacitor_SMD:C_0805_2012Metric_Pad1.18x1.45mm_HandSolder, F.Cu at (128.5, 105.8)
- added C43: 4.7uF, Capacitor_SMD:C_0805_2012Metric_Pad1.18x1.45mm_HandSolder, F.Cu at (140.2, 108.0)
- added C44: 22uF, Capacitor_SMD:C_0805_2012Metric_Pad1.18x1.45mm_HandSolder, F.Cu at (114.7, 124.0)
- added C45: 4.7uF, Capacitor_SMD:C_0805_2012Metric_Pad1.18x1.45mm_HandSolder, F.Cu at (114.7, 126.0)
- added C46: 22uF, Capacitor_SMD:C_0805_2012Metric_Pad1.18x1.45mm_HandSolder, F.Cu at (124.1, 124.3)
- added C47: 4.7uF, Capacitor_SMD:C_0805_2012Metric_Pad1.18x1.45mm_HandSolder, F.Cu at (128.1, 124.3)
- added C48: 1uF, Capacitor_SMD:C_0805_2012Metric_Pad1.18x1.45mm_HandSolder, F.Cu at (134.4, 124.3)
- added C49: 22uF, Capacitor_SMD:C_0805_2012Metric_Pad1.18x1.45mm_HandSolder, F.Cu at (140.2, 113.0)
- added C50: 4.7uF, Capacitor_SMD:C_0805_2012Metric_Pad1.18x1.45mm_HandSolder, F.Cu at (140.2, 115.6)
- added C51: 470nF, Capacitor_SMD:C_0805_2012Metric_Pad1.18x1.45mm_HandSolder, F.Cu at (140.2, 110.5)
- added C52: 220nF, Capacitor_SMD:C_0603_1608Metric_Pad1.08x0.95mm_HandSolder, F.Cu at (129.4, 98.8)
- added C53: 1uF, Capacitor_SMD:C_0805_2012Metric_Pad1.18x1.45mm_HandSolder, F.Cu at (125.7, 105.8)
- added C54: 220nF, Capacitor_SMD:C_0805_2012Metric_Pad1.18x1.45mm_HandSolder, F.Cu at (119.6, 105.8)
- added C55: 1uF, Capacitor_SMD:C_0805_2012Metric_Pad1.18x1.45mm_HandSolder, F.Cu at (121.7, 105.8)
- added C56: 22uF, Capacitor_SMD:C_0805_2012Metric_Pad1.18x1.45mm_HandSolder, F.Cu at (106.2, 114.4)
- added C57: 22uF, Capacitor_SMD:C_0805_2012Metric_Pad1.18x1.45mm_HandSolder, F.Cu at (108.3, 114.4)
- added C58: 22uF, Capacitor_SMD:C_0805_2012Metric_Pad1.18x1.45mm_HandSolder, F.Cu at (106.2, 118.8)
- added C59: 22uF, Capacitor_SMD:C_0805_2012Metric_Pad1.18x1.45mm_HandSolder, F.Cu at (108.3, 118.8)
- added C60: 22uF, Capacitor_SMD:C_0805_2012Metric_Pad1.18x1.45mm_HandSolder, F.Cu at (121.0, 131.6)
- added C61: 22uF, Capacitor_SMD:C_0805_2012Metric_Pad1.18x1.45mm_HandSolder, F.Cu at (121.0, 129.5)
- added C62: 22uF, Capacitor_SMD:C_0805_2012Metric_Pad1.18x1.45mm_HandSolder, F.Cu at (139.4, 120.6)
- added C63: 22uF, Capacitor_SMD:C_0805_2012Metric_Pad1.18x1.45mm_HandSolder, F.Cu at (137.4, 120.6)
- added C64: 22uF, Capacitor_SMD:C_0805_2012Metric_Pad1.18x1.45mm_HandSolder, F.Cu at (131.6, 104.8)
- added C65: 22uF, Capacitor_SMD:C_0805_2012Metric_Pad1.18x1.45mm_HandSolder, F.Cu at (131.6, 106.9)
- added C66: 10nF, Capacitor_SMD:C_0805_2012Metric_Pad1.18x1.45mm_HandSolder, F.Cu at (131.6, 102.7)
- added C67: 10uF, Capacitor_SMD:C_0805_2012Metric_Pad1.18x1.45mm_HandSolder, F.Cu at (136.3, 111.0)
- added C68: 1uF, Capacitor_SMD:C_0805_2012Metric_Pad1.18x1.45mm_HandSolder, F.Cu at (91.2, 108.0)
- added C69: 10uF, Capacitor_SMD:C_0805_2012Metric_Pad1.18x1.45mm_HandSolder, F.Cu at (91.2, 115.6)
- added C70: 47uF, Capacitor_SMD:C_0805_2012Metric_Pad1.18x1.45mm_HandSolder, F.Cu at (147.6, 110.5)
- added C71: 47uF, Capacitor_SMD:C_0805_2012Metric_Pad1.18x1.45mm_HandSolder, F.Cu at (147.6, 108.0)
- added C72: 22uF, Capacitor_SMD:C_0805_2012Metric_Pad1.18x1.45mm_HandSolder, F.Cu at (144.1, 105.4)
- added C73: 22uF, Capacitor_SMD:C_0805_2012Metric_Pad1.18x1.45mm_HandSolder, F.Cu at (144.1, 102.9)
- added D16: MBR120LSFT3G, Diode_SMD:D_SOD-123F, F.Cu at (129.4, 111.3)
- added D17: PGOOD, LED_SMD:LED_0805_2012Metric_Pad1.15x1.40mm_HandSolder, F.Cu at (91.2, 133.3)
- added D18: FAULT, LED_SMD:LED_0805_2012Metric_Castellated, F.Cu at (85.1, 133.3)
- added D19: D, Diode_SMD:D_0805_2012Metric_Pad1.15x1.40mm_HandSolder, F.Cu at (153.0, 104.1)
- added D20: D, Diode_SMD:D_0805_2012Metric_Pad1.15x1.40mm_HandSolder, F.Cu at (153.0, 101.6)
- added D21: D, Diode_SMD:D_0805_2012Metric_Pad1.15x1.40mm_HandSolder, F.Cu at (153.0, 127.0)
- added D22: D, Diode_SMD:D_0805_2012Metric_Pad1.15x1.40mm_HandSolder, F.Cu at (153.0, 116.8)
- added D23: D, Diode_SMD:D_0805_2012Metric_Pad1.15x1.40mm_HandSolder, F.Cu at (153.0, 132.1)
- added D24: D, Diode_SMD:D_0805_2012Metric_Pad1.15x1.40mm_HandSolder, F.Cu at (153.0, 129.5)
- added D25: D, Diode_SMD:D_0805_2012Metric_Pad1.15x1.40mm_HandSolder, F.Cu at (153.0, 124.5)
- added D26: D, Diode_SMD:D_0805_2012Metric_Pad1.15x1.40mm_HandSolder, F.Cu at (153.0, 121.9)
- added D27: D, Diode_SMD:D_0805_2012Metric_Pad1.15x1.40mm_HandSolder, F.Cu at (153.0, 106.7)
- added D28: D, Diode_SMD:D_0805_2012Metric_Pad1.15x1.40mm_HandSolder, F.Cu at (153.0, 119.4)
- added D29: D, Diode_SMD:D_0805_2012Metric_Pad1.15x1.40mm_HandSolder, F.Cu at (153.0, 111.8)
- added D30: D, Diode_SMD:D_0805_2012Metric_Pad1.15x1.40mm_HandSolder, F.Cu at (153.0, 109.2)
- added D31: D, Diode_SMD:D_0805_2012Metric_Pad1.15x1.40mm_HandSolder, F.Cu at (153.0, 114.3)
- added J12: Conn_01x02, Connector_PinHeader_2.54mm:PinHeader_1x02_P2.54mm_Vertical, F.Cu at (86.4, 109.2)
- added J13: Conn_01x03, Connector_PinHeader_2.54mm:PinHeader_1x03_P2.54mm_Vertical, F.Cu at (116.8, 96.5)
- added J14: Conn_01x03, Connector_PinHeader_2.54mm:PinHeader_1x03_P2.54mm_Vertical, F.Cu at (94.0, 124.5)
- added J15: Barrel_Jack_Switch, Connector_BarrelJack:BarrelJack_Horizontal, F.Cu at (95.2, 97.3)
- added J16: Conn_01x03, Connector_PinHeader_2.54mm:PinHeader_1x03_P2.54mm_Vertical, F.Cu at (86.4, 116.8)
- added J17: Conn_01x03, Connector_PinHeader_2.54mm:PinHeader_1x03_P2.54mm_Vertical, F.Cu at (99.1, 129.5)
- added J18: Conn_01x03, Connector_PinHeader_2.54mm:PinHeader_1x03_P2.54mm_Vertical, F.Cu at (106.7, 129.5)
- added J19: Conn_01x02, Connector_PinHeader_2.54mm:PinHeader_1x02_P2.54mm_Vertical, F.Cu at (99.1, 104.9)
- added J20: Conn_01x03, Connector_PinHeader_2.54mm:PinHeader_1x03_P2.54mm_Vertical, F.Cu at (106.7, 101.6)
- added J21: Conn_02x13_Odd_Even, Connector_PinHeader_2.54mm:PinHeader_2x13_P2.54mm_Vertical, F.Cu at (170.2, 101.6)
- added J22: Conn_01x03, Connector_PinHeader_2.54mm:PinHeader_1x03_P2.54mm_Vertical, F.Cu at (146.7, 97.2)
- added J23: Conn_01x06, Connector_PinHeader_2.54mm:PinHeader_1x06_P2.54mm_Vertical, F.Cu at (101.6, 124.5)
- added L10: 2.2uH, Inductor_SMD:L_1008_2520Metric_Pad1.43x2.20mm_HandSolder, F.Cu at (133.1, 112.0)
- added L6: 1.5uH, Inductor_SMD:L_1008_2520Metric_Pad1.43x2.20mm_HandSolder, F.Cu at (110.9, 114.4)
- added L7: 1.5uH, Inductor_SMD:L_1008_2520Metric_Pad1.43x2.20mm_HandSolder, F.Cu at (110.9, 118.7)
- added L8: 1.5uH, Inductor_SMD:L_1008_2520Metric_Pad1.43x2.20mm_HandSolder, F.Cu at (120.9, 126.9)
- added L9: 1.5uH, Inductor_SMD:L_1008_2520Metric_Pad1.43x2.20mm_HandSolder, F.Cu at (134.1, 118.3)
- added NT1: Net-Tie_2, TinyNetTies:NetTie-2_SMD_Pad0.254mm, F.Cu at (110.8, 121.9)
- added NT10: Net-Tie_2, TinyNetTies:NetTie-2_SMD_Pad0.254mm, F.Cu at (141.2, 101.6)
- added NT11: Net-Tie_2, TinyNetTies:NetTie-2_SMD_Pad0.254mm, F.Cu at (117.8, 118.8)
- added NT12: Net-Tie_2, TinyNetTies:NetTie-2_SMD_Pad0.254mm, F.Cu at (127.8, 118.5)
- added NT13: Net-Tie_2, TinyNetTies:NetTie-2_SMD_Pad0.254mm, F.Cu at (125.7, 109.8)
- added NT14: Net-Tie_2, TinyNetTies:NetTie-2_SMD_Pad0.254mm, F.Cu at (117.8, 114.2)
- added NT2: Net-Tie_2, TinyNetTies:NetTie-2_SMD_Pad0.254mm, F.Cu at (117.2, 129.0)
- added NT3: Net-Tie_2, TinyNetTies:NetTie-2_SMD_Pad0.254mm, F.Cu at (125.6, 121.8)
- added NT4: Net-Tie_2, TinyNetTies:NetTie-2_SMD_Pad0.254mm, F.Cu at (112.6, 114.9)
- added NT5: Net-Tie_2, TinyNetTies:NetTie-2_SMD_Pad0.254mm, F.Cu at (118.4, 129.2)
- added NT6: Net-Tie_2, TinyNetTies:NetTie-2_SMD_Pad0.254mm, F.Cu at (112.6, 118.2)
- added NT7: Net-Tie_2, TinyNetTies:NetTie-2_SMD_Pad0.254mm, F.Cu at (142.2, 118.3)
- added NT8: Net-Tie_2, TinyNetTies:NetTie-2_SMD_Pad0.254mm, F.Cu at (126.7, 111.1)
- added NT9: Net-Tie_2, TinyNetTies:NetTie-2_SMD_Pad0.254mm, F.Cu at (122.9, 110.7)
- added Q1: FDMA908PZ, Package_TO_SOT_SMD:Vishay_PowerPAK_SC70-6L_Single, F.Cu at (146.7, 114.3)
- added Q2: Q_PMOS_GSD, Package_TO_SOT_SMD:SOT-23, F.Cu at (90.9, 129.5)
- added Q3: Q_PMOS_GSD, Package_TO_SOT_SMD:SOT-23, F.Cu at (85.1, 129.5)
- added R20: 4K7, Resistor_SMD:R_0805_2012Metric_Pad1.20x1.40mm_HandSolder, B.Cu at (101.6, 100.1)
- added R21: 4K7, Resistor_SMD:R_0805_2012Metric_Pad1.20x1.40mm_HandSolder, B.Cu at (103.6, 100.1)
- added R22: 100K, Resistor_SMD:R_0805_2012Metric_Pad1.20x1.40mm_HandSolder, B.Cu at (100.6, 137.2)
- added R23: 100K, Resistor_SMD:R_0805_2012Metric_Pad1.20x1.40mm_HandSolder, B.Cu at (97.8, 119.4)
- added R24: 100K, Resistor_SMD:R_0805_2012Metric_Pad1.20x1.40mm_HandSolder, B.Cu at (105.1, 137.2)
- added R25: 100K, Resistor_SMD:R_0805_2012Metric_Pad1.20x1.40mm_HandSolder, B.Cu at (97.8, 114.3)
- added R26: 100K, Resistor_SMD:R_0805_2012Metric_Pad1.20x1.40mm_HandSolder, B.Cu at (97.8, 111.8)
- added R27: 2K2, Resistor_SMD:R_0805_2012Metric_Pad1.20x1.40mm_HandSolder, F.Cu at (91.2, 135.6)
- added R28: 2K2, Resistor_SMD:R_0805_2012Metric_Pad1.20x1.40mm_HandSolder, F.Cu at (85.1, 135.6)
- added R29: 2K2, Resistor_SMD:R_0805_2012Metric_Pad1.20x1.40mm_HandSolder, F.Cu at (160.0, 104.1)
- added R30: 2K2, Resistor_SMD:R_0805_2012Metric_Pad1.20x1.40mm_HandSolder, F.Cu at (160.0, 101.6)
- added R31: 2K2, Resistor_SMD:R_0805_2012Metric_Pad1.20x1.40mm_HandSolder, F.Cu at (160.0, 127.0)
- added R32: 2K2, Resistor_SMD:R_0805_2012Metric_Pad1.20x1.40mm_HandSolder, F.Cu at (160.0, 116.8)
- added R33: 2K2, Resistor_SMD:R_0805_2012Metric_Pad1.20x1.40mm_HandSolder, F.Cu at (160.0, 132.1)
- added R34: 2K2, Resistor_SMD:R_0805_2012Metric_Pad1.20x1.40mm_HandSolder, F.Cu at (160.0, 129.5)
- added R35: 2K2, Resistor_SMD:R_0805_2012Metric_Pad1.20x1.40mm_HandSolder, F.Cu at (160.0, 124.5)
- added R36: 2K2, Resistor_SMD:R_0805_2012Metric_Pad1.20x1.40mm_HandSolder, F.Cu at (160.0, 121.9)
- added R37: 2K2, Resistor_SMD:R_0805_2012Metric_Pad1.20x1.40mm_HandSolder, F.Cu at (160.0, 106.7)
- added R38: 2K2, Resistor_SMD:R_0805_2012Metric_Pad1.20x1.40mm_HandSolder, F.Cu at (160.0, 119.4)
- added R39: 2K2, Resistor_SMD:R_0805_2012Metric_Pad1.20x1.40mm_HandSolder, F.Cu at (160.0, 111.8)
- added R40: 2K2, Resistor_SMD:R_0805_2012Metric_Pad1.20x1.40mm_HandSolder, F.Cu at (160.0, 109.2)
- added R41: 2K2, Resistor_SMD:R_0805_2012Metric_Pad1.20x1.40mm_HandSolder, F.Cu at (160.0, 114.3)
- added SW5: SW_SPST, Button_Switch_SMD:SW_Push_1P1T_NO_CK_KMR2, F.Cu at (105.2, 106.2)
- added TP15: TestPoint, TestPoint:TestPoint_Pad_D1.0mm, F.Cu at (166.4, 104.1)
- added TP16: TestPoint, TestPoint:TestPoint_Pad_D1.0mm, F.Cu at (166.4, 101.6)
- added TP17: TestPoint, TestPoint:TestPoint_Pad_D1.0mm, F.Cu at (166.4, 127.0)
- added TP18: TestPoint, TestPoint:TestPoint_Pad_D1.0mm, F.Cu at (166.4, 116.8)
- added TP19: TestPoint, TestPoint:TestPoint_Pad_D1.0mm, F.Cu at (166.4, 132.1)
- added TP20: TestPoint, TestPoint:TestPoint_Pad_D1.0mm, F.Cu at (166.4, 129.5)
- added TP21: TestPoint, TestPoint:TestPoint_Pad_D1.0mm, F.Cu at (166.4, 124.5)
- added TP22: TestPoint, TestPoint:TestPoint_Pad_D1.0mm, F.Cu at (166.4, 121.9)
- added TP23: TestPoint, TestPoint:TestPoint_Pad_D1.0mm, F.Cu at (166.4, 106.7)
- added TP24: TestPoint, TestPoint:TestPoint_Pad_D1.0mm, F.Cu at (166.4, 119.4)
- added TP25: TestPoint, TestPoint:TestPoint_Pad_D1.0mm, F.Cu at (166.4, 111.8)
- added TP26: TestPoint, TestPoint:TestPoint_Pad_D1.0mm, F.Cu at (166.4, 109.2)
- added TP27: TestPoint, TestPoint:TestPoint_Pad_D1.0mm, F.Cu at (166.4, 114.3)
- added U2: PF3000, Package_DFN_QFN:QFN-48-1EP_7x7mm_P0.5mm_EP5.3x5.3mm_ThermalVias, F.Cu at (122.7, 115.6)
- added U3: SE8233X2, Package_TO_SOT_SMD:SOT-23, F.Cu at (91.2, 111.8)
- C12, C13, C14, C15, C16: footprint Capacitor_SMD:C_0603_1608Metric_Pad1.08x0.95mm_HandSolder -> Capacitor_SMD:C_0805_2012Metric_Pad1.18x1.45mm_HandSolder
- D1, D2: footprint Diode_SMD:D_0805_2012Metric_Pad1.15x1.40mm_HandSolder -> LED_SMD:LED_0805_2012Metric_Pad1.15x1.40mm_HandSolder
- moved C24 0.25 mm to (125.0, 53.1)
- moved C15 0.13 mm to (131.3, 69.1)
Connections:
- net /STPMIC1_Board/sheet60878B3D/SCL renamed /STPMIC1_Board/SCL
- net /STPMIC1_Board/sheet60878B3D/SDA renamed /STPMIC1_Board/SDA
Routing:
- net /STPMIC1_Board/VBUCK3: track 26.9 -> 169.5 mm
- net GNDS: track 82.1 -> 217.5 mm, vias 38 -> 66
- net /PF3000_Board/VSNVS_OUT: track 0.00 -> 117.7 mm, vias 0 -> 1
- net /PF3000_Board/SW1B_OUT: track 0.00 -> 106.2 mm, vias 0 -> 1
- net /PF3000_Board/SW1A_OUT: track 0.00 -> 92.8 mm, vias 0 -> 1
- net /PF3000_Board/LDO1_OUT: track 0.00 -> 89.2 mm, vias 0 -> 1
- net /STPMIC1_Board/VBUCK2: track 19.9 -> 106.2 mm
- net /PF3000_Board/LDO2_OUT: track 0.00 -> 84.0 mm, vias 0 -> 1
- net /PF3000_Board/SW2_OUT: track 0.00 -> 81.6 mm, vias 0 -> 2
- net /PF3000_Board/SW3_OUT: track 0.00 -> 79.6 mm, vias 0 -> 3
- net /PF3000_Board/VPWR: track 0.00 -> 70.3 mm
- net /STPMIC1_Board/VBUCK1: track 17.1 -> 86.0 mm
- net /PF3000_Board/SWBST_OUT: track 0.00 -> 67.4 mm, vias 0 -> 1
- net /PF3000_Board/LDO3_OUT: track 0.00 -> 66.2 mm, vias 0 -> 1
- net /PF3000_Board/LDO4_OUT: track 0.00 -> 61.7 mm, vias 0 -> 1
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- added copper zone on SmallSignal+Power.Cu, net /PF3000_Board/SW2_OUT
- added copper zone on SmallSignal+Power.Cu, net /PF3000_Board/VIN
- added copper zone on SmallSignal+Power.Cu, net /PF3000_Board/V_PU
- added copper zone on SmallSignal+Power.Cu, net /STPMIC1_Board/SWIN_Ext
- added copper zone on SmallSignal+Power.Cu, net /STPMIC1_Board/VBAT
- added copper zone on SmallSignal+Power.Cu, net /STPMIC1_Board/VIO
- added copper zone on SmallSignal+Power.Cu, net /STPMIC1_Board/sheet60878B3D/VSWIN
- added copper zone on Ground.Cu, net GNDS
- removed copper zone on In2.Cu, net /STPMIC1_Board/SWIN_Ext
- removed copper zone on In1.Cu, net /STPMIC1_Board/VBAT
- removed copper zone on In2.Cu, net /STPMIC1_Board/VBOOST
- removed copper zone on In2.Cu, net /STPMIC1_Board/VBUCK1
- removed copper zone on In2.Cu, net /STPMIC1_Board/VBUCK2
- removed copper zone on In2.Cu, net /STPMIC1_Board/VBUCK3
- removed copper zone on In2.Cu, net /STPMIC1_Board/VBUCK4
- removed copper zone on In2.Cu, net /STPMIC1_Board/VIO
- removed copper zone on In2.Cu, net /STPMIC1_Board/VLDO1
- removed copper zone on In2.Cu, net /STPMIC1_Board/VLDO2
- removed copper zone on In2.Cu, net /STPMIC1_Board/VLDO3
- removed copper zone on In2.Cu, net /STPMIC1_Board/VLDO4
- removed copper zone on In2.Cu, net /STPMIC1_Board/VLDO5
- removed copper zone on In2.Cu, net /STPMIC1_Board/VLDO6
- removed copper zone on In2.Cu, net /STPMIC1_Board/VOTG
- removed copper zone on In2.Cu, net /STPMIC1_Board/VREFDDR
- removed copper zone on In2.Cu, net /STPMIC1_Board/VSWOUT
- removed copper zone on In2.Cu, net /STPMIC1_Board/sheet60878B3D/VSWIN
- removed copper zone on F.Cu, net GNDS
Other:
- board text added: "BUCK1A"
- board text added: "BUCK1B"
- board text added: "INTB"
- board text added: "MAX 3V"
- board text added: "PWRON"
- board text added: "RESET BMCU"
- board text added: "SDSEL"
- board text added: "SD_VSEL"
- board text added: "STDBY"
- board text added: "V33"
- board text added: "VCCSD"
- board text added: "VCOREDIG"
- board text added: "VDBG"
- board text added: "VDDIO"
- board text added: "VDDOTP"
- board text added: "VDOG"
- board text added: "VIN"
- board text added: "VPU"
- board text added: "VPWR"
- board text added: "VREFDDR"
- board text added: "VSNVS"
- board text added: "V_PU"

Commit message: updated RevA Layout
Parts:
- C10, C11, C17, C18, C19, C21, C22, C25, C8, C9: footprint Capacitor_SMD:C_0603_1608Metric_Pad1.08x0.95mm_HandSolder -> Capacitor_SMD:C_0805_2012Metric_Pad1.18x1.45mm_HandSolder
- C68, C69, Q2, Q3, R27, R28, U3: moved to B.Cu
- J4: value USB_B_Micro -> Barrel_Jack; footprint Connector_USB:USB_Micro-B_Molex-105017-0001 -> Connector_BarrelJack:BarrelJack_Horizontal
- moved D1 18.5 mm to (115.4, 89.2), turned to 180 degrees
- moved C70 14.4 mm to (146.0, 124.8)
- moved C71 14.2 mm to (146.0, 122.1)
- moved R1 14.1 mm to (110.5, 89.2)
- moved SW5 13.7 mm to (92.6, 111.6), turned to 270 degrees
- moved C1 11.7 mm to (102.9, 87.4)
- moved J4 10.8 mm to (95.2, 84.6), turned to 0 degrees
- moved J1 6.58 mm to (86.4, 73.7)
- moved C68 5.24 mm to (94.5, 112.0), turned to 90 degrees
- moved J15 3.05 mm to (95.2, 100.3)
- moved J12 2.79 mm to (86.4, 112.0)
- moved J19 2.65 mm to (101.6, 104.1)
- moved C17 2.60 mm to (134.8, 72.4)
- moved J18 2.54 mm to (104.1, 129.5)
- moved C8 2.35 mm to (132.8, 72.4)
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Connections:
- J15 pad 3: /PF3000_Board/VPWR -> Net-(J15-Pad3)
- J4 pad 2: Net-(J4-Pad2) -> GNDS
- J4 pad 3: Net-(J4-Pad3) -> (no net)
Routing:
- net /STPMIC1_Board/VIO: track 12.8 -> 48.2 mm
- net /STPMIC1_Board/VBOOST: track 61.1 -> 93.2 mm
- net /STPMIC1_Board/sheet60878B3D/VSWIN: track 9.80 -> 31.1 mm
- net /STPMIC1_Board/VBUCK3: track 169.5 -> 188.2 mm
- net /STPMIC1_Board/VBAT: track 71.4 -> 87.4 mm
- net /PF3000_Board/V_PU: track 12.2 -> 27.2 mm, vias 5 -> 3
- net Net-(J4-Pad6): track 12.4 -> 0.00 mm
- net /PF3000_Board/PWRON: track 31.5 -> 42.4 mm
- net Net-(C70-Pad2): track 21.3 -> 31.3 mm
- net GNDS: track 217.5 -> 211.0 mm, vias 66 -> 62
- net /STPMIC1_Board/VIO_Ext: track 0.00 -> 5.33 mm
- net /PF3000_Board/VDDIO: track 55.8 -> 60.1 mm
- net /PF3000_Board/VDBG: track 10.3 -> 7.16 mm
- net /STPMIC1_Board/VLDO6: track 62.0 -> 64.7 mm
- net /PF3000_Board/RESETBMCU: track 42.8 -> 45.4 mm, vias 1 -> 0
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- removed copper zone on F.Cu, net /STPMIC1_Board/VBOOST
- removed copper zone on F.Cu, net /STPMIC1_Board/VBUCK3
- removed copper zone on F.Cu, net /STPMIC1_Board/VIO
- removed copper zone on F.Cu, net /STPMIC1_Board/VIO_Ext
- removed copper zone on F.Cu, net /STPMIC1_Board/sheet60878B3D/VSWIN
Other:
- board text added: "3.3V"
- board text added: "< 1.85V"
- board text added: "> 2.85V"
- board text added: "BYPASS MEM"
- board text added: "DEEP SLEEP MODE"
- board text added: "DISABLE VPWR"
- board text added: "ENABLE VPWR"
- board text added: "FAULT"
- board text added: "OFF"
- board text added: "ON"
- board text added: "OTP"
- board text added: "PGOOD"
- board text added: "POWER ENABLE"
- board text added: "USE MEM"
- board text added: "VCC_SD OUTPUT RANGE"
- board text removed: "SDSEL"
- board text removed: "VCOREDIG"
- board text removed: "VDDOTP"
- board text removed: "VDOG"
- board text removed: "VPU"
- board text removed: "VPWR"

Commit message: Completed RevA
Parts:
- added JP1: Jumper_NO_Small, Jumper:SolderJumper-2_P1.3mm_Open_RoundedPad1.0x1.5mm, B.Cu at (90.4, 126.6)
- added JP2: Jumper_NO_Small, Jumper:SolderJumper-2_P1.3mm_Open_RoundedPad1.0x1.5mm, B.Cu at (85.1, 126.6)
- BT1: footprint Battery:BatteryHolder_Seiko_MS621F -> Panasonic_ML_series:ML1220_F1BN
- C1: footprint Capacitor_SMD:C_Elec_4x5.4 -> Capacitor_SMD:C_Elec_6.3x7.7
- C2, C20, C23, C3, C4, C5, C52, C6, C7: footprint Capacitor_SMD:C_0603_1608Metric_Pad1.08x0.95mm_HandSolder -> Capacitor_SMD:C_0805_2012Metric_Pad1.18x1.45mm_HandSolder
- D10, D11, D12, D13, D14, D15, D19, D20, D21, D22, D23, D24, D25, D26, D27, D28, D29, D3, D30, D31, D4, D5, D6, D7, D8, D9: footprint Diode_SMD:D_0805_2012Metric_Pad1.15x1.40mm_HandSolder -> LED_SMD:LED_0805_2012Metric_Pad1.15x1.40mm_HandSolder
- L10: footprint Inductor_SMD:L_1008_2520Metric_Pad1.43x2.20mm_HandSolder -> Inductor_SMD:L_Coilcraft_LPS4018
- Q2, Q3: moved to F.Cu
- moved R20 15.2 mm to (115.1, 93.0), turned to 90 degrees
- moved R21 11.8 mm to (113.0, 93.0), turned to 270 degrees
- moved BT1 10.2 mm to (136.7, 89.7), turned to 90 degrees
- moved J13 8.42 mm to (125.2, 97.3), turned to 270 degrees
- moved J23 8.13 mm to (101.6, 116.3)
- moved R25 8.13 mm to (97.8, 106.2)
- moved R26 8.13 mm to (97.8, 103.6)
- moved C52 7.42 mm to (136.7, 100.5), turned to 180 degrees
- moved J8 7.39 mm to (112.5, 79.4), turned to 0 degrees
- moved J17 7.37 mm to (106.4, 129.5)
- moved J19 7.00 mm to (103.0, 97.3), turned to 90 degrees
- moved R22 6.79 mm to (106.2, 137.2), turned to 0 degrees
- moved J2 6.14 mm to (87.1, 48.3), turned to 180 degrees
- moved J20 5.68 mm to (110.4, 97.3), turned to 90 degrees
- moved C7 3.18 mm to (131.2, 51.9)
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Connections:
- Q2 pad 2: /PF3000_Board/V_PU -> /PF3000_Board/VDBG
- Q3 pad 2: /PF3000_Board/V_PU -> /PF3000_Board/VDBG
Routing:
- net /PF3000_Board/VDBG: track 7.16 -> 41.1 mm, vias 0 -> 1
- net /PF3000_Board/VDDIO: track 60.1 -> 91.4 mm, vias 1 -> 2
- net /PF3000_Board/INTB: track 49.3 -> 73.9 mm, vias 0 -> 1
- net /STPMIC1_Board/sheet60878B3D/VSWIN: track 31.1 -> 46.7 mm
- net /STPMIC1_Board/VBUCK2: track 106.2 -> 121.2 mm
- net /STPMIC1_Board/VBUCK3: track 188.2 -> 201.5 mm
- net /PF3000_Board/PWRON: track 42.4 -> 51.6 mm
- net /PF3000_Board/V_PU: track 27.2 -> 18.4 mm
- net /PF3000_Board/SDA: track 29.2 -> 20.8 mm
- net /STPMIC1_Board/VIO_Ext: track 5.33 -> 13.2 mm
- net /PF3000_Board/RESETBMCU: track 45.4 -> 52.2 mm, vias 0 -> 2
- net /PF3000_Board/SD_VSEL: track 41.7 -> 48.2 mm
- net /STPMIC1_Board/SWIN_Ext: track 0.00 -> 5.08 mm
- net /STPMIC1_Board/VBAT: track 87.4 -> 92.3 mm
- net /PF3000_Board/STANDBY: track 41.7 -> 45.9 mm
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- removed copper zone on SmallSignal+Power.Cu, net /STPMIC1_Board/SWIN_Ext
- removed copper zone on SmallSignal+Power.Cu, net /STPMIC1_Board/sheet60878B3D/VSWIN
Other:
- board text added: "(I2C)"
- board text added: "3V"
- board text added: "Chris Sutton RevA 1021"
- board text added: "DISABLE"
- board text added: "ENABLE"
- board text added: "EXT SWIN"
- board text added: "EXT VIO"
- board text added: "LDO3 IN"
- board text added: "NO MEM"
- board text added: "PF3000"
- board text added: "PMIC DEV BOARD"
- board text added: "PWR"
- board text added: "STPMIC1"
- board text removed: "BUCK 3"
- board text removed: "BYPASS MEM"
- board text removed: "EXT"
- board text removed: "MAX 3V"
- board text removed: "PWR CTL"
- board text removed: "SELECT LDO3 IN"
- board text removed: "SWIN EXT"
- board text removed: "SWIN INPUT"
- board text removed: "VIO EXT"
- board text removed: "VIO INPUT"
